File: BatteryBox.kicad_sch (KiCad schematic)
At the start: 33 parts, among them J1 Conn_01x02, J10 Conn_01x02, J11 Conn_01x02, J12 Conn_01x02, J13 Conn_01x02, J14 Conn_01x02, J15 Conn_01x02, J2 Conn_01x02, J3 Conn_01x02, J4 Conn_01x04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

Commit message: Finalising PCB layout. Needs final component puchase and footprint check.
Connections:
- net GND: now also K1.8; no longer K1.1
- net at J13.1 (Pin_1), J14.1 (Pin_1), J15.1 (Pin_1): no longer K1.6
- net at D2.2 (A), D4.1 (K), M1.3 (Out+): now also K1.1; no longer K1.4, K1.8
- net at K1.2: no longer K2.4
Other:
- moved on the sheet: K1
Changed lines of the file:
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@@
     (pin "2")
   )
-  (symbol (lib_name "SANYOU_SRD_Form_C_1") (lib_id "Relay:SANYOU_SRD_Form_C") (at 114.3 40.64 90) (mirror x) (unit 1)
-    (in_bom yes) (on_board yes)
-    (property "Reference" "K1" (id 0) (at 125.73 40.64 90))
-    (property "Value" "SANYOU_SRD_Form_C" (id 1) (at 127 40.64 90)
-      (effects (font (size 1.27 1.27)) hide)
-    )
-    (property "Footprint" "Relay_THT:Relay_SPDT_Panasonic_JW1_FormC" (id 2) (at 125.73 41.91 0)
+  (symbol (lib_name "SANYOU_SRD_Form_C_1") (lib_id "Relay:SANYOU_SRD_Form_C") (at 114.3 40.64 270) (unit 1)
+    (in_bom yes) (on_board yes)
+    (property "Reference" "K1" (id 0) (at 102.87 40.64 90))
+    (property "Value" "SANYOU_SRD_Form_C" (id 1) (at 101.6 40.64 90)
+      (effects (font (size 1.27 1.27)) hide)
+    )
+    (property "Footprint" "Relay_THT:Relay_SPDT_Panasonic_JW1_FormC" (id 2) (at 102.87 41.91 0)
       (effects (font (size 1.27 1.27)) (justify left) hide)
     )
@@
       (effects (font (size 1.27 1.27)) hide)
     )
+    (pin "1")
+    (pin "2")
+    (pin "4")
     (pin "6")
-    (pin "1")
-    (pin "4")
-    (pin "2")
     (pin "8")
   )
@@
       (effects (font (size 1.27 1.27)) hide)
     )
+    (pin "1")
+    (pin "2")
+    (pin "4")
     (pin "6")
-    (pin "1")
-    (pin "4")
-    (pin "2")
     (pin "8")
   )
